Commit message: 基于 V3.2 补齐 J7 舵机与双指联动 URDF
从 V3.2 装配体生成专用 FCStd 快照，继续排除 A000、B000，原始 STEP 保留在仓库外。补齐七个舵机和双 finger，增加基于 CAD 推定的反向 mimic 关节，并同步七轴预览、渲染图、来源记录和下载包。

验证：113 个保留源实体唯一归属；9 个连杆、7 个控制关节及 1 个从动关节；25 份网格校验、独立 URDF 解析、J7 联动计算、零位与开合姿态渲染、文档检查及 ZIP 完整性通过。本轮浏览器界面未自动验收；实机限位、零位及传动关系仍待确认。

File: hardware/robot-description/touch_r1_description/urdf/touch-r1.urdf (robot description, URDF)
Before this commit: robot touch_r1_leader_arm_preview, 7 links, 6 joints
Links:
- added link left_finger; visual mesh filename=../meshes/left_finger-finger.stl
- added link right_finger; visual mesh filename=../meshes/right_finger-finger.stl; visual mesh filename=../meshes/right_finger-horn.stl
- link link_6: geometry visual mesh filename=../meshes/link_6-horn.stl; visual mesh filename=../meshes/link_6-servo.stl
Joints:
- added joint joint_7: type continuous, parent link_6, child right_finger, origin xyz=0.006675 0.0541 0.00235 rpy=0 0 0, axis -0 -1 0
- added joint left_finger_joint: type continuous, parent link_6, child left_finger, origin xyz=-0.015325 0.0541 0.00235 rpy=0 0 0, axis 0 -1 0, mimic joint=joint_7 multiplier=-1.0 offset=0.0
- joint joint_3: axis 1 2.2e-09 0 -> 1 0 0; origin xyz=-9.99997e-05 -0.165625 0 rpy=0 0 0 -> xyz=-0.0001 -0.165625 0 rpy=0 0 0
- joint joint_4: axis 1 2.2e-09 0 -> 1 0 0; origin xyz=0.0003623925 0.165625 0.03875 rpy=0 0 0 -> xyz=0.0003623929 0.165625 0.03875 rpy=0 0 0
- joint joint_5: origin xyz=-0.0002311965 0.048745 0.019343455 rpy=0 0 0 -> xyz=-0.0002311964 0.048745 0.019343455 rpy=0 0 0
- joint joint_6: axis 2.2e-09 -1 0 -> -0 -1 0
